Commit message: Removed pa10-7c (in a fork branch now) and left/right references

File: urdf/pa10-7a.urdf.xacro (robot description, xacro)
@@ -1,15 +1,14 @@
 <?xml version="1.0"?>
-<robot name="PA10c"
+<robot name="PA10-7a"
 		 xmlns:xacro="http://www.ros.org/wiki/xacro"
 		 xmlns:sensor="http://playerstage.sourceforge.net/gazebo/xmlschema/#sensor"
 		 xmlns:controller="http://playerstage.sourceforge.net/gazebo/xmlschema/#controller"
        xmlns:interface="http://playerstage.sourceforge.net/gazebo/xmlschema/#interface">
-  <xacro:include filename="../urdf/util.urdf.xacro"/>
-  <xacro:macro name="pa10c_arm" params="name kinematic:=false">
+  <xacro:macro name="pa10_7a_arm" params="name kinematic:=false">
   <link name="${name}arm_base_link">
     <visual>
       <origin xyz="0 0 0" rpy="0 0 0"/>
       <geometry>
-        <mesh filename="package://pa10_7a_description/meshes/pa-7c/link0_mesh.dae" scale="1 1 1" />
+        <mesh filename="package://pa10_7a_description/meshes/link0_mesh.dae" scale="1 1 1" />
       </geometry>
     </visual>
@@ -17,17 +16,17 @@
       <origin xyz="0 0 0.100" rpy="0 0 0"/>
       <geometry>
-        <cylinder length="0.200" radius="0.115"/>
-      </geometry>
-    </collision>
-    <collision>
-      <origin xyz="0 0.130 0.090" rpy="0 0 0"/>
-      <geometry>
-        <box size="0.160 0.080 0.160" />
-      </geometry>
-    </collision>
-    <inertial>
-      <mass value="6.88" />
-      <origin xyz="0 0 0.091" rpy="0 0 0"/>
-      <inertia ixx="0.043" ixy="0" ixz="0" iyy="0.043" iyz="0" izz="0.0416"/>
+		  <cylinder length="0.20" radius="0.115"/>
+      </geometry>
+    </collision>
+    <collision>
+       <origin xyz="0 0.120 0.060" rpy="0 0 0"/>
+      <geometry>
+        <box size="0.130 0.060 0.060" />
+      </geometry>
+    </collision>
+    <inertial>
+      <mass value="3.04" />
+      <origin xyz="0 0 0.075" rpy="0 0 0"/>
+      <inertia ixx="0.0193" ixy="0" ixz="0" iyy="0.0193" iyz="0" izz="0.0184"/>
     </inertial>
   </link>
@@ -41,5 +40,5 @@
       <origin xyz="0 0 0" rpy="0 0 0"/>
       <geometry>
-        <mesh filename="package://pa10_7a_description/meshes/pa-7c/link1_mesh.dae" scale="1 1 1" />
+        <mesh filename="package://pa10_7a_description/meshes/link1_mesh.dae" scale="1 1 1" />
       </geometry>
     </visual>
@@ -51,5 +50,5 @@
     </collision>
     <collision>
-      <origin xyz="0.0 0.105 0.3" rpy="0 0 0"/>
+      <origin xyz="0.0 0.104 0.298" rpy="0 0 0"/>
       <geometry>
 		  <box size="0.140 0.05 0.180" />
@@ -57,5 +56,5 @@
     </collision>
     <collision>
-      <origin xyz="0.0 -0.105 0.3" rpy="0 0 0"/>
+      <origin xyz="0.0 -0.104 0.298" rpy="0 0 0"/>
       <geometry>
 		  <box size="0.140 0.05 0.180" />
@@ -63,7 +62,7 @@
     </collision>
     <inertial>
-      <mass value="7.33" />
-      <origin xyz="0 0 0.160" rpy="0 0 0"/>
-      <inertia ixx="0.11" ixy="0" ixz="0" iyy="0.11" iyz="0" izz="0.037"/>
+      <mass value="9.78" />
+      <origin xyz="0 0 0.148" rpy="0 0 0"/>
+      <inertia ixx="0.145" ixy="0" ixz="0" iyy="0.145" iyz="0" izz="0.049"/>
     </inertial>
   </link>
@@ -73,11 +72,11 @@
   <link name="${name}arm_2_link">
     <visual>
-      <origin xyz="0 0 -0.317" rpy="0 0 0"/>
-      <geometry>
-        <mesh filename="package://pa10_7a_description/meshes/pa-7c/link2_mesh.dae" scale="1 1 1" />
-      </geometry>
-    </visual>
-    <collision>
-      <origin xyz="0 0 0.183" rpy="0 0 0"/>
+      <origin xyz="0 0 -0.315" rpy="0 0 3.1415"/>
+      <geometry>
+        <mesh filename="package://pa10_7a_description/meshes/link2_mesh.dae" scale="1 1 1" />
+      </geometry>
+    </visual>
+    <collision>
+      <origin xyz="0 0 0.181" rpy="0 0 0"/>
       <geometry>
         <cylinder length="0.266" radius="0.07"/>
@@ -91,7 +90,7 @@
     </collision>
     <inertial>
-      <mass value="10.76" />
-      <origin xyz="0 0 0.063" rpy="0 0 0"/>
-      <inertia ixx="0.168" ixy="0" ixz="0" iyy="0.168" iyz="0" izz="0.026"/>
+      <mass value="8.41" />
+      <origin xyz="0 0 0.06325" rpy="0 0 0"/>
+      <inertia ixx="0.1316" ixy="0" ixz="0" iyy="0.1316" iyz="0" izz="0.0206"/>
     </inertial>
   </link>
@@ -101,17 +100,17 @@
   <link name="${name}arm_3_link">
     <visual>
-      <origin xyz="0 0 -0.317" rpy="0 0 0"/>
-      <geometry>
-        <mesh filename="package://pa10_7a_description/meshes/pa-7c/link3_mesh.dae" scale="1 1 1" />
-      </geometry>
-    </visual>
-    <collision>
-      <origin xyz="0 0 0.333" rpy="0 0 0"/>
-      <geometry>
-         <box size="0.120 0.116 0.034" />
-      </geometry>
-    </collision>
-    <collision>
-      <origin xyz="0.0 0.083 0.413" rpy="0 0 0"/>
+      <origin xyz="0 0 -0.315" rpy="0 0 0"/>
+      <geometry>
+        <mesh filename="package://pa10_7a_description/meshes/link3_mesh.dae" scale="1 1 1" />
+      </geometry>
+    </visual>
+    <collision>
+      <origin xyz="0 0 0.336" rpy="0 0 0"/>
+      <geometry>
+         <box size="0.120 0.116 0.044" />
+      </geometry>
+    </collision>
+    <collision>
+      <origin xyz="0.0 0.083 0.411" rpy="0 0 0"/>
       <geometry>
 		  <box size="0.120 0.05 0.20" />
@@ -119,5 +118,5 @@
     </collision>
     <collision>
-      <origin xyz="0.0 -0.083 0.413" rpy="0 0 0"/>
+      <origin xyz="0.0 -0.083 0.411" rpy="0 0 0"/>
       <geometry>
 		  <box size="0.120 0.05 0.20" />
@@ -125,7 +124,7 @@
     </collision>
     <inertial>
-      <mass value="2.97" />
-      <origin xyz="0 0 0.346" rpy="0 0 0"/>
-      <inertia ixx="0.028" ixy="0" ixz="0" iyy="0.028" iyz="0" izz="0.073"/>
+      <mass value="3.51" />
+      <origin xyz="0 0 0.3605" rpy="0 0 0"/>
+      <inertia ixx="0.0298" ixy="0" ixz="0" iyy="0.0298" iyz="0" izz="0.009"/>
     </inertial>
   </link>
@@ -135,11 +134,11 @@
   <link name="${name}arm_4_link">
     <visual>
-      <origin xyz="0 0 -0.767" rpy="0 0 0"/>
-      <geometry>
-        <mesh filename="package://pa10_7a_description/meshes/pa-7c/link4_mesh.dae" scale="1 1 1" />
-      </geometry>
-    </visual>
-    <collision>
-      <origin xyz="0 0 0.170" rpy="0 0 0"/>
+      <origin xyz="0 0 -0.765" rpy="0 0 0"/>
+      <geometry>
+        <mesh filename="package://pa10_7a_description/meshes/link4_mesh.dae" scale="1 1 1" />
+      </geometry>
+    </visual>
+    <collision>
+      <origin xyz="0 0 0.150" rpy="0 0 0"/>
       <geometry>
         <cylinder length="0.248" radius="0.055"/>
@@ -153,7 +152,7 @@
     </collision>
     <inertial>
-      <mass value="4.86" />
-      <origin xyz="0 0 0.0485" rpy="0 0 0"/>
-      <inertia ixx="0.0055" ixy="0" ixz="0" iyy="0.0055" iyz="0" izz="0.0073"/>
+      <mass value="4.31" />
+      <origin xyz="0 0 0.04609" rpy="0 0 0"/>
+      <inertia ixx="0.0493" ixy="0" ixz="0" iyy="0.0493" iyz="0" izz="0.0065"/>
     </inertial>
   </link>
@@ -163,31 +162,31 @@
   <link name="${name}arm_5_link">
     <visual>
-      <origin xyz="0 0 -0.767" rpy="0 0 0"/>
-      <geometry>
-        <mesh filename="package://pa10_7a_description/meshes/pa-7c/link5_mesh.dae" scale="1 1 1" />
-      </geometry>
-    </visual>
-    <collision>
-      <origin xyz="0 0 0.322" rpy="0 0 0"/>
-      <geometry>
-         <box size="0.09 0.102 0.070" />
-      </geometry>
-    </collision>
-    <collision>
-      <origin xyz="0.0 0.066 0.403" rpy="0 0 0"/>
-      <geometry>
-		  <box size="0.09 0.03 0.242" />
-      </geometry>
-    </collision>
-    <collision>
-      <origin xyz="0.0 -0.066 0.403" rpy="0 0 0"/>
-      <geometry>
-		  <box size="0.09 0.03 0.242" />
-      </geometry>
-    </collision>
-    <inertial>
-      <mass value="3.08" />
-      <origin xyz="0 0 0.368" rpy="0 0 0"/>
-      <inertia ixx="0.02" ixy="0" ixz="0" iyy="0.02" iyz="0" izz="0.0046"/>
+      <origin xyz="0 0 -0.765" rpy="0 0 0"/>
+      <geometry>
+        <mesh filename="package://pa10_7a_description/meshes/link5_mesh.dae" scale="1 1 1" />
+      </geometry>
+    </visual>
+    <collision>
+      <origin xyz="0 0 0.300" rpy="0 0 0"/>
+      <geometry>
+         <box size="0.09 0.082 0.070" />
+      </geometry>
+    </collision>
+    <collision>
+      <origin xyz="0.0 0.051 0.401" rpy="0 0 0"/>
+      <geometry>
+		  <box size="0.09 0.03 0.284" />
+      </geometry>
+    </collision>
+    <collision>
+      <origin xyz="0.0 -0.051 0.401" rpy="0 0 0"/>
+      <geometry>
+		  <box size="0.09 0.03 0.284" />
+      </geometry>
+    </collision>
+    <inertial>
+      <mass value="3.45" />
+      <origin xyz="0 0 0.335" rpy="0 0 0"/>
+      <inertia ixx="0.0486" ixy="0" ixz="0" iyy="0.0486" iyz="0" izz="0.0052"/>
     </inertial>
   </link>
@@ -197,19 +196,19 @@
   <link name="${name}arm_6_link">
     <visual>
-      <origin xyz="0 0 -1.247" rpy="0 0 0"/>
-      <geometry>
-        <mesh filename="package://pa10_7a_description/meshes/pa-7c/link6_mesh.dae" scale="1 1 1" />
-      </geometry>
-    </visual>
-    <collision>
-      <origin xyz="0 0 -0.023" rpy="0 0 0"/>
-      <geometry>
-        <cylinder length="0.186" radius="0.05"/>
-      </geometry>
-    </collision>
-    <inertial>
-      <mass value="3.00" />
-      <origin xyz="0 0 -0.042" rpy="0 0 0"/>
-      <inertia ixx="0.011" ixy="0" ixz="0" iyy="0.011" iyz="0" izz="0.0038"/>
+      <origin xyz="0 0 -1.265" rpy="0 0 0"/>
+      <geometry>
+        <mesh filename="package://pa10_7a_description/meshes/link6_mesh.dae" scale="1 1 1" />
+      </geometry>
+    </visual>
+    <collision>
+      <origin xyz="0 0 -0.043" rpy="0 0 0"/>
+      <geometry>
+        <cylinder length="0.230" radius="0.035"/>
+      </geometry>
+    </collision>
+    <inertial>
+      <mass value="1.46" />
+      <origin xyz="0 0 -0.03" rpy="0 0 0"/>
+      <inertia ixx="0.0071" ixy="0" ixz="0" iyy="0.0071" iyz="0" izz="0.0015"/>
     </inertial>
   </link>
@@ -219,7 +218,7 @@
   <link name="${name}arm_7_link">
     <visual>
-      <origin xyz="0 0 0" rpy="0 0 0"/>
-      <geometry>
-        <mesh filename="package://pa10_7a_description/meshes/pa-7c/link7_mesh.dae" scale="1 1 1" />
+      <origin xyz="0 0 1.345" rpy="0 0 0"/>
+      <geometry>
+        <mesh filename="package://pa10_7a_description/meshes/link7_mesh.dae" scale="1 1 1" />
       </geometry>
     </visual>
@@ -227,11 +226,11 @@
       <origin xyz="0 0 -0.01" rpy="0 0 0"/>
       <geometry>
-        <cylinder length="0.02" radius="0.04"/>
-      </geometry>
-    </collision>
-    <inertial>
-      <mass value="0.12" />
-      <origin xyz="0 0 -0.048" rpy="0 0 0"/>
-      <inertia ixx="0.000052" ixy="0.0" ixz="0" iyy="0.000052" iyz="0" izz="0.000096"/>
+        <cylinder length="0.02" radius="0.035"/>
+      </geometry>
+    </collision>
+    <inertial>
+      <mass value="0.24" />
+      <origin xyz="0 0 -0.029" rpy="0 0 0"/>
+      <inertia ixx="0.0001" ixy="0" ixz="0" iyy="0.0001" iyz="0" izz="0.0002"/>
     </inertial>
   </link>
@@ -259,7 +258,7 @@
     <parent link="${name}arm_1_link"/>
     <child  link="${name}arm_2_link"/>
-    <origin xyz="0 0 0.317" rpy="0 0 0 "/>
+    <origin xyz="0 0 0.315" rpy="0 0 0 "/>
     <axis   xyz="0 1 0"/>
-    <limit lower="${-94/180*pi}" upper="${+94/180*pi}" effort="100" velocity="1" />
+    <limit lower="${-91/180*pi}" upper="${+91/180*pi}" effort="100" velocity="1" />
     <dynamics damping="0.2" friction="0" />
   </joint>
@@ -327,5 +326,5 @@
     <parent link="${name}arm_5_link"/>
     <child  link="${name}arm_6_link"/>
-    <origin xyz="0 0 0.480" rpy="0 0 0 "/>
+    <origin xyz="0 0 0.5" rpy="0 0 0 "/>
     <axis   xyz="0 1 0"/>
     <limit lower="${-165/180*pi}" upper="${165/180*pi}" effort="100" velocity="6.28" />
@@ -345,10 +344,10 @@
     <parent link="${name}arm_6_link"/>
     <child  link="${name}arm_7_link"/>
-    <origin xyz="0 0 0.07" rpy="0 0 0 "/>
+    <origin xyz="0 0 0.08" rpy="0 0 0 "/>
     <axis   xyz="0 0 1"/>
-    <limit lower="${-255/180*pi}" upper="${255/180*pi}" effort="100" velocity="6.28" />
-    <dynamics damping="0.2" friction="0" />
-  </joint>
-  <gazebo reference="${name}W2">
+    <limit lower="${-359/180*pi}" upper="${359/180*pi}" effort="100" velocity="6.28" />
+    <dynamics damping="0.2" friction="0" />
+  </joint>
+  <gazebo reference="${name}W1">
     <provideFeedback>1</provideFeedback>
     <implicitSpringDamper>1</implicitSpringDamper>
@@ -364,5 +363,5 @@
   </joint>
   <link name="${name}tool_mount" />
-   <gazebo reference="${name}tool_mount">
+  <gazebo reference="${name}tool_mount">
     <kinematic>${kinematic}</kinematic>
   </gazebo>
