Commit message: Changed controller plugin to gazebo_ros_control (get rid of shadow dependency) Added stand-alone launch

File: robots/pa10_7a_arm.urdf.xacro (robot description, xacro)
@@ -2,5 +2,5 @@
 <robot name="pa10-7a" xmlns:xacro="http://www.ros.org/wiki/xacro" >
   <xacro:include filename="$(find pa10_7a_description)/urdf/pa10-7a.urdf.xacro"/>
-  <xacro:include filename="$(find pa10_7a_description)/urdf/pa10_shadow_controller_manager.xacro"/>
+  <xacro:include filename="$(find pa10_7a_description)/urdf/pa10_ros_controller_manager.xacro"/>
   <link name="world" />
   <joint name="world_pa10_arm_base_joint" type="fixed">
@@ -10,4 +10,4 @@
   </joint>
   <xacro:pa10_7a_arm name="" />
-  <xacro:pa10_shadow_gazebo_controller_manager namespace="" />
+  <xacro:pa10_gazebo_ros_controller_manager namespace="" />
 </robot>

File: urdf/pa10-7a.urdf.xacro (robot description, xacro)
@@ -250,7 +250,11 @@
     <implicitSpringDamper>1</implicitSpringDamper>
   </gazebo>
-  <transmission type="sr_mechanism_model/SimpleTransmission" name="${name}S1_transmission">
-    <actuator name="${name}S1_actuator" />
+  <transmission name="${name}S1_transmission">
+    <type>transmission_interface/SimpleTransmission</type>
+    <actuator name="${name}S1_actuator">
+      <mechanicalReduction>1</mechanicalReduction>
+    </actuator>
     <joint name="${name}S1">
+      <hardwareInterface>PositionJointInterface</hardwareInterface>
     </joint>
   </transmission>
@@ -267,7 +271,11 @@
     <implicitSpringDamper>1</implicitSpringDamper>
   </gazebo>
-  <transmission type="sr_mechanism_model/SimpleTransmission" name="${name}S2_transmission">
-    <actuator name="${name}S2_actuator" />
+  <transmission name="${name}S2_transmission">
+    <type>transmission_interface/SimpleTransmission</type>
+    <actuator name="${name}S2_actuator">
+      <mechanicalReduction>1</mechanicalReduction>
+    </actuator>
     <joint name="${name}S2">
+      <hardwareInterface>PositionJointInterface</hardwareInterface>
     </joint>
   </transmission>
@@ -284,7 +292,11 @@
     <implicitSpringDamper>1</implicitSpringDamper>
   </gazebo>
-  <transmission type="sr_mechanism_model/SimpleTransmission" name="${name}S3_transmission">
-    <actuator name="${name}S3_actuator" />
+  <transmission name="${name}S3_transmission">
+    <type>transmission_interface/SimpleTransmission</type>
+    <actuator name="${name}S3_actuator">
+      <mechanicalReduction>1</mechanicalReduction>
+    </actuator>
     <joint name="${name}S3">
+      <hardwareInterface>PositionJointInterface</hardwareInterface>
     </joint>
   </transmission>
@@ -301,7 +313,11 @@
     <implicitSpringDamper>1</implicitSpringDamper>
   </gazebo>
-  <transmission type="sr_mechanism_model/SimpleTransmission" name="${name}E1_transmission">
-    <actuator name="${name}E1_actuator" />
+  <transmission name="${name}E1_transmission">
+    <type>transmission_interface/SimpleTransmission</type>
+    <actuator name="${name}E1_actuator">
+      <mechanicalReduction>1</mechanicalReduction>
+    </actuator>
     <joint name="${name}E1">
+      <hardwareInterface>PositionJointInterface</hardwareInterface>
     </joint>
   </transmission>
@@ -318,7 +334,11 @@
     <implicitSpringDamper>1</implicitSpringDamper>
   </gazebo>
-  <transmission type="sr_mechanism_model/SimpleTransmission" name="${name}E2_transmission">
-    <actuator name="${name}E2_actuator" />
+  <transmission name="${name}E2_transmission">
+    <type>transmission_interface/SimpleTransmission</type>
+    <actuator name="${name}E2_actuator">
+      <mechanicalReduction>1</mechanicalReduction>
+    </actuator>
     <joint name="${name}E2">
+      <hardwareInterface>PositionJointInterface</hardwareInterface>
     </joint>
   </transmission>
@@ -335,8 +355,11 @@
     <implicitSpringDamper>1</implicitSpringDamper>
   </gazebo>
-  <!-- <transmission type="transmission_interface/SimpleTransmission" name="${name}W1_transmission"> -->
-  <transmission type="sr_mechanism_model/SimpleTransmission" name="${name}W1_transmission">
-    <actuator name="${name}W1_actuator" />
+  <transmission name="${name}W1_transmission">
+    <type>transmission_interface/SimpleTransmission</type>
+    <actuator name="${name}W1_actuator">
+      <mechanicalReduction>1</mechanicalReduction>
+    </actuator>
     <joint name="${name}W1">
+      <hardwareInterface>PositionJointInterface</hardwareInterface>
     </joint>
   </transmission>
@@ -353,7 +376,11 @@
     <implicitSpringDamper>1</implicitSpringDamper>
   </gazebo>
-  <transmission type="sr_mechanism_model/SimpleTransmission" name="${name}W2_transmission">
-    <actuator name="${name}W2_actuator" />
+  <transmission name="${name}W2_transmission">
+    <type>transmission_interface/SimpleTransmission</type>
+    <actuator name="${name}W2_actuator">
+      <mechanicalReduction>1</mechanicalReduction>
+    </actuator>
     <joint name="${name}W2">
+      <hardwareInterface>PositionJointInterface</hardwareInterface>
     </joint>
   </transmission>

File: urdf/pa10_ros_controller_manager.xacro (robot description, xacro)
@@ -4,10 +4,9 @@
        xmlns:controller="http://playerstage.sourceforge.net/gazebo/xmlschema/#controller"
        xmlns:interface="http://playerstage.sourceforge.net/gazebo/xmlschema/#interface">
-	<!-- namespace must be set up according to launch file namespace -->
-  <xacro:macro name="pa10_shadow_gazebo_controller_manager" params="namespace">
+  <!-- namespace must be set up according to launch file namespace -->
+  <xacro:macro name="pa10_gazebo_ros_controller_manager" params="namespace">
 		<gazebo>
-			<plugin name="sr_gazebo_ros_controller_manager" filename="libsr_gazebo_ros_controller_manager.so">
-				<alwaysOn>true</alwaysOn>
-				<updateRate>1400.0</updateRate>
+			<plugin name="gazebo_ros_control" filename="libgazebo_ros_control.so">
+        <controlPeriod>0.001</controlPeriod>
 				<robotNamespace>${namespace}</robotNamespace>
 			</plugin>
